Commit message: added files for moveit

File: turtlebot_arm_description/urdf/arm_4dof.xacro (robot description, xacro)
@@ -61,5 +61,5 @@
     </bioloid_F3_fixed>
     <!-- gripper -->
-    <!-- <dynamixel_AX12_fixed parent="arm_joint4_frame2_link" name="gripper_servo">
+    <dynamixel_AX12_fixed parent="arm_joint4_frame2_link" name="gripper_servo">
       <origin xyz="0.01475 0 ${-AX12_WIDTH/2}" rpy="0 ${M_PI/2} 0"/>
     </dynamixel_AX12_fixed>
@@ -82,5 +82,5 @@
         <origin xyz=" 0 0 0 " rpy="0 0 0" />
         <geometry>
-          <mesh filename="package://turtlebot_arm_description/meshes/gripper_left.dae" scale="1 1 1"/>
+          <mesh filename="package://turtlebot_arm_description/meshes/gripper_left.dae"/>
         </geometry>
         <material name="${color}"/>

Commit message: added a gripper

File: turtlebot_arm_description/urdf/arm_4dof.xacro (robot description, xacro)
@@ -67,5 +67,5 @@
       <origin xyz="0 0 0" rpy="0 0 0"/>
       <axis xyz="0 1 0"/>
-      <limit effort="30" velocity="0.785" lower="-0.40" upper="0.46" />
+      <limit effort="30" velocity="0.785" lower="-0.40" upper="1.27" />
       <parent link="gripper_servo_link"/>
       <child link="gripper_active_link" />
@@ -76,9 +76,9 @@
         <origin xyz="0 0 0" />
         <inertia ixx="1.0" ixy="0.0" ixz="0.0"
-          iyy="1.0" iyz="0.0"
-          izz="1.0" />
+                           iyy="1.0" iyz="0.0"
+                                     izz="1.0" />
       </inertial>
       <visual>
-        <origin xyz=" 0 0 0 " rpy="0 0 0" />
+        <origin xyz=" 0 0 0 " rpy="${-M_PI/2} 0 0" />
         <geometry>
           <mesh filename="package://turtlebot_arm_description/meshes/gripper_left.dae"/>
@@ -92,5 +92,35 @@
         </geometry>
       </collision>
-    </link> -->
+    </link>
+    <joint name="gripper_mimic_joint" type="revolute">
+      <mimic joint="gripper_joint" multiplier="-1.0" offset="0"/>
+      <origin xyz="0 0 -0.04" rpy="0 0 0"/>
+      <axis xyz="0 1 0"/>
+      <limit effort="30" velocity="0.785" lower="-0.40" upper="1.27" />
+      <parent link="gripper_servo_link"/>
+      <child link="gripper_mimic_link"/>
+    </joint>
+    <link name="gripper_mimic_link">
+      <inertial>
+        <mass value="0.00001" />
+        <origin xyz="0 0 0" />
+        <inertia ixx="1.0" ixy="0.0" ixz="0.0"
+                           iyy="1.0" iyz="0.0"
+                                     izz="1.0" />
+      </inertial>
+      <visual>
+        <origin xyz="0 0 0" rpy="${-M_PI/2} 0 0" />
+        <geometry>
+          <mesh filename="package://turtlebot_arm_description/meshes/gripper_right.dae"/>
+        </geometry>
+        <material name="${color}"/>
+      </visual>
+      <collision>
+        <origin xyz="0.0 0.0 0.00775" rpy="0 0 0" />
+        <geometry>
+          <box size="0.025 0.0485 0.0375"/>
+        </geometry>
+      </collision>
+    </link>
   </xacro:macro>
 </robot>

Commit message: modified the options of gripper model

File: turtlebot_arm_description/urdf/arm_4dof.xacro (robot description, xacro)
@@ -21,5 +21,5 @@
     <!-- shoulder pan joint -->
     <dynamixel_AX12_fixed parent="arm_base_link" name="arm_joint1_servo">
-      <origin xyz="0 0 0" rpy="${M_PI/2} 0 ${M_PI/2}"/>
+      <origin xyz="0 0 ${AX12_WIDTH/2}" rpy="${M_PI/2} 0 ${M_PI/2}"/>
     </dynamixel_AX12_fixed>
     <bioloid_F2_pan_revolute parent="arm_joint1_servo_link" name="arm_joint1_frame1" color="${color}"
@@ -84,10 +84,9 @@
           <mesh filename="package://turtlebot_arm_description/meshes/gripper_left.dae"/>
         </geometry>
-        <material name="${color}"/>
       </visual>
       <collision>
-        <origin xyz="0.0 0.0 0.00775" rpy="0 0 0" />
+        <origin xyz="0.0 0.0 0.02" rpy="0 0 0" />
         <geometry>
-          <box size="0.025 0.0485 0.0375"/>
+          <box size="0.025 0.048 0.06"/>
         </geometry>
       </collision>
@@ -114,10 +113,9 @@
           <mesh filename="package://turtlebot_arm_description/meshes/gripper_right.dae"/>
         </geometry>
-        <material name="${color}"/>
       </visual>
       <collision>
-        <origin xyz="0.0 0.0 0.00775" rpy="0 0 0" />
+        <origin xyz="0.0 0.0 -0.02" rpy="0 0 0" />
         <geometry>
-          <box size="0.025 0.0485 0.0375"/>
+          <box size="0.025 0.048 0.06"/>
         </geometry>
       </collision>

Commit message: modified the gripper's description for moveit

File: turtlebot_arm_description/urdf/arm_4dof.xacro (robot description, xacro)
@@ -60,4 +60,13 @@
       <origin xyz="0 0.008 ${F2_HEIGHT}" rpy="0 ${M_PI} ${-M_PI/2}" />
     </bioloid_F3_fixed>
+    <!-- gripper link joint (fake) -->
+    <joint name="gripper_link_joint" type="revolute">
+      <origin xyz="-0.005 0 -0.06" rpy="0 0 0" />
+      <parent link="arm_joint4_frame2_link"/>
+      <child link="gripper_link" />
+      <limit effort="30" velocity="1" lower="${-M_PI}" upper="${M_PI}"/>
+      <axis xyz="1 0 0"/>
+    </joint>
+    <link name="gripper_link" />
     <!-- gripper -->
     <dynamixel_AX12_fixed parent="arm_joint4_frame2_link" name="gripper_servo">

Commit message: added the example for IK and FK

File: turtlebot_arm_description/urdf/arm_4dof.xacro (robot description, xacro)
@@ -62,6 +62,6 @@
     <!-- gripper link joint (fake) -->
     <joint name="gripper_link_joint" type="revolute">
-      <origin xyz="-0.005 0 -0.06" rpy="0 0 0" />
-      <parent link="arm_joint4_frame2_link"/>
+      <origin xyz="0 0 0.1" rpy="0 -1.57 0" />
+      <parent link="arm_joint4_frame1_link"/>
       <child link="gripper_link" />
       <limit effort="30" velocity="1" lower="${-M_PI}" upper="${M_PI}"/>
@@ -105,5 +105,5 @@
       <origin xyz="0 0 -0.04" rpy="0 0 0"/>
       <axis xyz="0 1 0"/>
-      <limit effort="30" velocity="0.785" lower="-0.40" upper="1.27" />
+      <limit effort="30" velocity="0.785" lower="-1.27" upper="0.40" />
       <parent link="gripper_servo_link"/>
       <child link="gripper_mimic_link"/>

File: turtlebot_arm_description/urdf/arm_4dof_hardware.xacro (robot description, xacro)
@@ -219,5 +219,5 @@
     <joint name="${name}_joint" type="revolute">
       <insert_block name="origin" />
-      <axis xyz="0 0 -1"/>
+      <axis xyz="0 0 1"/>
       <limit effort="30" velocity="${vlimit}" lower="${llimit}" upper="${ulimit}" />
       <parent link="${parent}"/>
